File: vaz_pi5_integration.kicad_sch (KiCad schematic)
At the start: 3 parts, among them J1 GPIO_Pi5

Commit message: Update VAZ 21011 + Raspberry Pi 5 integration schematic with detailed GPIO connections and control system enhancements
Parts:
- removed C1: 100nF
- removed J1: GPIO_Pi5
- removed R1: 10k
Other:
- note added: "+12V from vehicle battery"
- note added: "+3.3V for GPIO level shifting"
- note added: "+5V for Raspberry Pi (via buck converter)"
- note added: "CONNECTORS:"
- note added: "Fuel Level Sensor"
- note added: "GND - Common ground with vehicle"
- note added: "GPIO INPUTS:"
- note added: "GPIO OUTPUTS:"
- note added: "GPIO12 - Throttle Position (ADC)"
- note added: "GPIO13 - Brake Pressure (ADC)"
- note added: "GPIO14/GPIO15 - Serial Port for OBD-II Diagnostics"
- note added: "GPIO17 - Starter Relay"
- note added: "GPIO22 - Cooling Fan Relay"
- note added: "GPIO27 - Fuel Pump Relay"
- note added: "GPIO4 - Ignition Control"
- note added: "GPIO5 - RPM Sensor"
- note added: "GPIO6 - Speed Sensor"
- note added: "I2C Bus (GPIO2=SDA, GPIO3=SCL)"
- note added: "Oil Pressure Sensor"
- note added: "POWER SUPPLY:"
- note added: "Raspberry Pi 5 GPIO Connection Scheme"
- note added: "Temperature Sensor (DS18B20)"
- note added: "UART INTERFACE:"
- note removed: "GPIO Connections: - GPIO2/GPIO3: I2C (sensors) - GPIO4-GPIO27: Control outputs - GPIO14/GPIO15: UART (diagnostics) - GPIO10/GPIO9/GPIO11: SPI (optional)"
- note removed: "Raspberry Pi 5 GPIO Connections for VAZ 21011 Control"
- title: VAZ 21011 + Raspberry Pi 5 Integration -> VAZ 21011 + Raspberry Pi 5 Control System
Changed lines of the file:
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@@
   (paper "A4")
   (title_block
-    (title "VAZ 21011 + Raspberry Pi 5 Integration")
+    (title "VAZ 21011 + Raspberry Pi 5 Control System")
     (date "2025-10-20")
     (rev "1.0")
-    (comment 1 "Control system for VAZ 21011")
-    (comment 2 "Using Raspberry Pi 5")
+    (comment 1 "Raspberry Pi 5 Control System for VAZ 21011")
+    (comment 2 "GPIO connections for engine management")
   )
-  (junction (at 100 100) (diameter 0) (color 0 0 0 0))
-  (wire (pts (xy 50 100) (xy 100 100)) (stroke (width 0)))
-  (wire (pts (xy 100 100) (xy 150 100)) (stroke (width 0)))
-  (symbol (at 30 100 0)
-    (property "Reference" "J1" (id 0) (at 0 0 0))
-    (property "Value" "GPIO_Pi5" (id 1) (at 0 -2.54 0))
-    (pin "1")
+  (text "Raspberry Pi 5 GPIO Connection Scheme" (at 20 20 0)
+    (effects (font (size 2 2) (thickness 0.4)))
   )
-  (symbol (at 80 100 0)
-    (property "Reference" "R1" (id 0) (at 0 0 0))
-    (property "Value" "10k" (id 1) (at 0 -2.54 0))
-    (pin "1")
-    (pin "2")
+  (text "CONNECTORS:" (at 20 40 0)
+    (effects (font (size 1.5 1.5) (thickness 0.3)))
   )
-  (symbol (at 130 100 0)
-    (property "Reference" "C1" (id 0) (at 0 0 0))
-    (property "Value" "100nF" (id 1) (at 0 -2.54 0))
-    (pin "1")
-    (pin "2")
+  (text "I2C Bus (GPIO2=SDA, GPIO3=SCL)" (at 20 60 0)
+    (effects (font (size 1 1) (thickness 0.2)))
   )
-  (text "Raspberry Pi 5 GPIO Connections\nfor VAZ 21011 Control" (at 50 150 0)
-    (effects (font (size 1.27 1.27) (thickness 0.15)))
+  (text "Temperature Sensor (DS18B20)" (at 20 80 0)
+    (effects (font (size 1 1) (thickness 0.2)))
   )
-  (text "GPIO Connections:\n- GPIO2/GPIO3: I2C (sensors)\n- GPIO4-GPIO27: Control outputs\n- GPIO14/GPIO15: UART (diagnostics)\n- GPIO10/GPIO9/GPIO11: SPI (optional)" (at 50 130 0)
-    (effects (font (size 1.27 1.27) (thickness 0.15)))
+  (text "Fuel Level Sensor" (at 20 100 0)
+    (effects (font (size 1 1) (thickness 0.2)))
+  )
+  (text "Oil Pressure Sensor" (at 20 120 0)
+    (effects (font (size 1 1) (thickness 0.2)))
+  )
+  (text "GPIO OUTPUTS:" (at 20 150 0)
+    (effects (font (size 1.5 1.5) (thickness 0.3)))
+  )
+  (text "GPIO4 - Ignition Control" (at 20 170 0)
+    (effects (font (size 1 1) (thickness 0.2)))
+  )
+  (text "GPIO17 - Starter Relay" (at 20 190 0)
+    (effects (font (size 1 1) (thickness 0.2)))
+  )
+  (text "GPIO27 - Fuel Pump Relay" (at 20 210 0)
+    (effects (font (size 1 1) (thickness 0.2)))
+  )
+  (text "GPIO22 - Cooling Fan Relay" (at 20 230 0)
+    (effects (font (size 1 1) (thickness 0.2)))
+  )
+  (text "GPIO INPUTS:" (at 20 260 0)
+    (effects (font (size 1.5 1.5) (thickness 0.3)))
+  )
+  (text "GPIO5 - RPM Sensor" (at 20 280 0)
+    (effects (font (size 1 1) (thickness 0.2)))
+  )
+  (text "GPIO6 - Speed Sensor" (at 20 300 0)
+    (effects (font (size 1 1) (thickness 0.2)))
+  )
+  (text "GPIO12 - Throttle Position (ADC)" (at 20 320 0)
+    (effects (font (size 1 1) (thickness 0.2)))
+  )
+  (text "GPIO13 - Brake Pressure (ADC)" (at 20 340 0)
+    (effects (font (size 1 1) (thickness 0.2)))
+  )
+  (text "UART INTERFACE:" (at 20 370 0)
+    (effects (font (size 1.5 1.5) (thickness 0.3)))
+  )
+  (text "GPIO14/GPIO15 - Serial Port for OBD-II Diagnostics" (at 20 390 0)
+    (effects (font (size 1 1) (thickness 0.2)))
+  )
+  (text "POWER SUPPLY:" (at 250 40 0)
+    (effects (font (size 1.5 1.5) (thickness 0.3)))
+  )
+  (text "+12V from vehicle battery" (at 250 60 0)
+    (effects (font (size 1 1) (thickness 0.2)))
+  )
+  (text "+5V for Raspberry Pi (via buck converter)" (at 250 80 0)
+    (effects (font (size 1 1) (thickness 0.2)))
+  )
+  (text "+3.3V for GPIO level shifting" (at 250 100 0)
+    (effects (font (size 1 1) (thickness 0.2)))
+  )
+  (text "GND - Common ground with vehicle" (at 250 120 0)
+    (effects (font (size 1 1) (thickness 0.2)))
   )
 )
